File: kicad/LT1/LT1.kicad_pcb (KiCad board)
At the start: 2 copper layers, 160 parts, among them J1 USB_B_Micro, J2 Conn_01x05_Socket, J3 Conn_01x02_Socket, J4 Conn_01x02_Socket, Q1 2N7002K, Q10 2N7002K, Q11 2N7002K, Q12 2N7002K, Q13 2N7002K, Q14 2N7002K, Q15 2N7002K, Q16 2N7002K, Q17 2N7002K, Q18 2N7002K, Q19 2N7002K, Q2 2N7002K, Q20 2N7002K, Q21 2N7002K, Q22 2N7002K, Q23 2N7002K, Q24 2N7002K, Q25 2N7002K, Q26 2N7002K, Q27 2N7002K, Q28 2N7002K, Q29 2N7002K, Q3 2N7002K, Q30 2N7002K, Q31 2N7002K, Q32 2N7002K, Q4 2N7002K, Q5 2N7002K, Q6 2N7002K, Q7 2N7002K, Q8 2N7002K, Q9 2N7002K, SW1 SW_Push, SW2 SW_Push, SW3 SW_Push, SW4 SW_Push, SW5 SW_Push, SW6 SW_Push, SW7 SW_Push, U1 MCP73831-2-OT, U2 TLV75533PDBV, U4 74HC595D, U5 74HC595D, U6 74HC595D, U7 74HC595D, U8 MCP111T-xxxE_TT, U9 STM32L412C8Tx, Y1 32 kHz (ABS06)

Commit message: LT1 some routing and placing
Parts:
- removed TP10, TP11, TP12, TP13, TP14, TP15, TP16, TP17, TP4, TP5, TP6, TP7, TP8, TP9: TestPoint, TestPoint:TestPoint_Pad_D1.0mm
- added C17: 100nF, Capacitor_SMD:C_0603_1608Metric, B.Cu at (61.0, 98.0)
- added C18: 10uF, Capacitor_SMD:C_0805_2012Metric, B.Cu at (70.5, 70.5)
- added C19: 10uF, Capacitor_SMD:C_0805_2012Metric, B.Cu at (91.5, 70.5)
- BT1, D7, D8, J3, J4, Q31, Q32, R46, R47, R48, R49: moved to B.Cu
- C14: value 100nF -> 10nF
- moved R47 144.5 mm to (58.0, 73.0), turned to 180 degrees
- moved J4 144.3 mm to (65.0, 69.5), turned to -90 degrees
- moved D8 140.2 mm to (65.5, 72.5), turned to 180 degrees
- moved Q32 138.8 mm to (58.0, 70.0), turned to 90 degrees
- moved R49 135.2 mm to (61.5, 68.5)
- moved R46 132.9 mm to (79.0, 73.0), turned to 180 degrees
- moved D7 128.3 mm to (86.5, 72.5), turned to 180 degrees
- moved J3 127.6 mm to (86.0, 69.5), turned to -90 degrees
- moved Q31 127.1 mm to (79.0, 70.0), turned to 90 degrees
- moved R48 123.2 mm to (82.5, 68.5)
- moved J2 121.2 mm to (30.6, 83.1), turned to 0 degrees
- moved SW4 94.7 mm to (243.2, 135.2)
- moved TP18 91.9 mm to (72.5, 109.0), turned to 180 degrees
- moved TP19 91.8 mm to (70.0, 109.0), turned to 180 degrees
- moved BT1 80.4 mm to (40.4, 102.1), turned to 180 degrees
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Connections:
- TP1 pad 1: Net-(U9-PH0) -> ALM0
- TP18 pad 1: ALM0 -> Net-(U9-PB14)
- TP19 pad 1: ALM1 -> Net-(U9-PB15)
- TP2 pad 1: Net-(U9-PH1) -> ALM1
- U9 pad 27: ALM0 -> Net-(U9-PB14)
- U9 pad 28: ALM1 -> Net-(U9-PB15)
- U9 pad 5: Net-(U9-PH0) -> ALM1
- U9 pad 6: Net-(U9-PH1) -> ALM0
Routing:
- net BTN_PLAY: track 0.00 -> 267.5 mm, vias 0 -> 4
- net BTN_MODE: track 0.00 -> 249.3 mm, vias 0 -> 4
- net BTN_STOP: track 0.00 -> 235.7 mm, vias 0 -> 4
- net Net-(D1-R4-Pad12): track 0.00 -> 233.0 mm, vias 0 -> 3
- net Net-(D1-R3): track 0.00 -> 224.9 mm, vias 0 -> 1
- net Net-(D1-R1): track 0.00 -> 223.1 mm, vias 0 -> 3
- net Net-(D1-R2): track 0.00 -> 222.0 mm, vias 0 -> 3
- net Net-(D1-R7): track 0.00 -> 206.6 mm
- net BTN_UP4: track 0.00 -> 203.2 mm, vias 0 -> 4
- net Net-(D1-R6): track 0.00 -> 201.2 mm
- net Net-(D1-R5): track 0.00 -> 200.6 mm
- net DISP_COL_SRCLR: track 0.00 -> 190.0 mm, vias 0 -> 2
- net DISP_COL_SRCLK: track 0.00 -> 184.4 mm, vias 0 -> 2
- net DISP_COL_RCLK: track 0.00 -> 184.2 mm, vias 0 -> 2
- net DISP_COL_OE: track 0.00 -> 181.2 mm, vias 0 -> 2
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
Commit message: LT1 all routed, gerber exported
Parts:
- moved S1 10.2 mm to (233.3, 70.4), turned to -90 degrees
- moved C18 10.0 mm to (80.5, 69.5)
- moved C19 10.0 mm to (101.5, 69.5)
- moved D7 10.0 mm to (96.5, 71.5)
- moved D8 10.0 mm to (75.5, 71.5)
- moved J3 10.0 mm to (96.0, 68.5)
- moved J4 10.0 mm to (75.0, 68.5)
- moved Q31 10.0 mm to (89.0, 69.0)
- moved Q32 10.0 mm to (68.0, 69.0)
- moved R46 10.0 mm to (89.0, 72.0)
- moved R47 10.0 mm to (68.0, 72.0)
- moved R48 10.0 mm to (92.5, 67.5), turned to 180 degrees
- moved R49 10.0 mm to (71.5, 67.5), turned to 180 degrees
- moved TP1 10.0 mm to (92.0, 72.0)
- moved TP2 10.0 mm to (71.0, 72.0)
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Connections:
- D1 pad 11: Net-(Q3-D) -> Net-(D1-C3)
- D1 pad 12: Net-(D1-R4-Pad12) -> Net-(D1-R4)
- D1 pad 4: Net-(Q3-D) -> (no net)
- D1 pad 5: Net-(D1-R4-Pad12) -> (no net)
- D2 pad 11: Net-(Q8-D) -> Net-(D2-C3)
- D2 pad 12: Net-(D1-R4-Pad12) -> Net-(D1-R4)
- D2 pad 4: Net-(Q8-D) -> (no net)
- D2 pad 5: Net-(D1-R4-Pad12) -> (no net)
- D3 pad 11: Net-(Q13-D) -> Net-(D3-C3)
- D3 pad 12: Net-(D1-R4-Pad12) -> Net-(D1-R4)
- D3 pad 4: Net-(Q13-D) -> (no net)
- D3 pad 5: Net-(D1-R4-Pad12) -> (no net)
- D4 pad 11: Net-(Q18-D) -> Net-(D4-C3)
- D4 pad 12: Net-(D1-R4-Pad12) -> Net-(D1-R4)
- D4 pad 4: Net-(Q18-D) -> (no net)
- D4 pad 5: Net-(D1-R4-Pad12) -> (no net)
- D5 pad 11: Net-(Q23-D) -> Net-(D5-C3)
- D5 pad 12: Net-(D1-R4-Pad12) -> Net-(D1-R4)
- D5 pad 4: Net-(Q23-D) -> (no net)
- D5 pad 5: Net-(D1-R4-Pad12) -> (no net)
- D6 pad 11: Net-(Q28-D) -> Net-(D6-C3)
- D6 pad 12: Net-(D1-R4-Pad12) -> Net-(D1-R4)
- D6 pad 4: Net-(Q28-D) -> (no net)
- D6 pad 5: Net-(D1-R4-Pad12) -> (no net)
- Q13 pad 3: Net-(Q13-D) -> Net-(D3-C3)
- Q18 pad 3: Net-(Q18-D) -> Net-(D4-C3)
- Q23 pad 3: Net-(Q23-D) -> Net-(D5-C3)
- Q28 pad 3: Net-(Q28-D) -> Net-(D6-C3)
- Q3 pad 3: Net-(Q3-D) -> Net-(D1-C3)
- Q8 pad 3: Net-(Q8-D) -> Net-(D2-C3)
- R4 pad 2: Net-(D1-R4-Pad12) -> Net-(D1-R4)
Routing:
- net +3.3V: track 35.5 -> 384.8 mm, vias 1 -> 14
- net Net-(D1-R4-Pad12): track 233.0 -> 0.00 mm, vias 3 -> 0
- net Net-(D1-R4): track 0.00 -> 232.8 mm, vias 0 -> 3
- net SW0: track 7.63 -> 191.9 mm, vias 1 -> 2
- net SW1: track 5.00 -> 187.7 mm, vias 1 -> 2
- net SW2: track 6.28 -> 187.4 mm, vias 1 -> 2
- net SW3: track 7.85 -> 187.5 mm, vias 1 -> 2
- net SW4: track 8.06 -> 186.1 mm, vias 1 -> 2
- net Net-(Q3-D): track 72.6 -> 0.00 mm, vias 2 -> 0
- net Net-(D1-C3): track 0.00 -> 72.6 mm, vias 0 -> 3
- net Net-(D1-C2): track 28.3 -> 90.1 mm, vias 1 -> 2
- net Net-(Q8-D): track 54.5 -> 0.00 mm, vias 2 -> 0
- net Net-(D2-C3): track 0.00 -> 54.0 mm, vias 0 -> 2
- net Net-(D1-C5): track 18.8 -> 71.0 mm, vias 1 -> 2
- net nRST: track 4.48 -> 49.6 mm, vias 0 -> 4
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- added copper zone on B.Cu, net GND
- added copper zone on F.Cu, net GND
Other:
- board outline added: 245 x 76 mm
- board text added: "0"
- board text added: "164"
- board text added: "180"
- board text added: "266"
- board text added: "27"
- board text added: "78"
- board text removed: "50mil oder 100 mil Abstand"
