File: kicad/LT1/LT1Display.kicad_sch (KiCad schematic)
At the start: 81 parts, among them Q1 2N7002K, Q10 2N7002K, Q11 2N7002K, Q12 2N7002K, Q13 2N7002K, Q14 2N7002K, Q15 2N7002K, Q16 2N7002K, Q17 2N7002K, Q18 2N7002K, Q19 2N7002K, Q2 2N7002K, Q20 2N7002K, Q21 2N7002K, Q22 2N7002K, Q23 2N7002K, Q24 2N7002K, Q25 2N7002K, Q26 2N7002K, Q27 2N7002K, Q28 2N7002K, Q29 2N7002K, Q3 2N7002K, Q30 2N7002K, Q4 2N7002K, Q5 2N7002K, Q6 2N7002K, Q7 2N7002K, Q8 2N7002K, Q9 2N7002K, U4 74HC595, U5 74HC595, U6 74HC595, U7 74HC595

Commit message: LT1 started with PCB, added driver for piezo and vibra alarm
Parts:
- C1, C2, C3, C4: footprint (none) -> Capacitor_SMD:C_0603_1608Metric
- Q1, Q10, Q11, Q12, Q13, Q14, Q15, Q16, Q17, Q18, Q19, Q2, Q20, Q21, Q22, Q23, Q24, Q25, Q26, Q27, Q28, Q29, Q3, Q30, Q4, Q5, Q6, Q7, Q8, Q9: footprint Package_TO_SOT_SMD:SOT-23 -> Package_TO_SOT_SMD:TSOT-23
- R1, R10, R11, R12, R13, R14, R15, R16, R17, R18, R19, R2, R20, R21, R22, R23, R24, R25, R26, R27, R28, R29, R3, R30, R31, R32, R33, R34, R35, R36, R37, R4, R5, R6, R7, R8, R9: footprint (none) -> Resistor_SMD:R_0603_1608Metric
- U4, U5, U6, U7: value 74HC595 -> 74HC595D; footprint (none) -> Package_SO:SO-16_3.9x9.9mm_P1.27mm

Commit message: LT1 all routed, gerber exported
Connections:
- net at D4.11 (C3), Q13.3 (D): no longer D4.4 (C3)
- net at D1.11 (C3), Q28.3 (D): no longer D1.4 (C3)
- net at D1.12 (R4), D2.12 (R4), D3.12 (R4)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: no longer D1.5 (R4), D2.5 (R4), D3.5 (R4), D4.5 (R4), D5.5 (R4), D6.5 (R4)
- net at D2.11 (C3), Q23.3 (D): no longer D2.4 (C3)
- net at D5.11 (C3), Q8.3 (D): no longer D5.4 (C3)
- net at D3.11 (C3), Q18.3 (D): no longer D3.4 (C3)
- net at D6.11 (C3), Q3.3 (D): no longer D6.4 (C3)
Changed lines of the file:
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@@
     )
   )
-  (symbol (lib_id "TC20-11SRWA:TC20-11SRWA") (at 285.75 53.34 270) (unit 1)
+  (symbol (lib_name "TC20-11SRWA_1") (lib_id "TC20-11SRWA:TC20-11SRWA") (at 285.75 53.34 270) (unit 1)
     (in_bom yes) (on_board yes) (dnp no)
-    (property "Reference" "D1" (at 299.72 64.77 90)
+    (property "Reference" "D1" (at 278.13 64.77 90)
       (effects (font (size 1.27 1.27)) (justify right))
     )
-    (property "Value" "TC20-11SRWA" (at 274.32 58.42 0)
+    (property "Value" "TC20-11SRWA" (at 274.32 57.15 0)
       (effects (font (size 1.27 1.27)) (justify right))
     )
@@
     (pin "2")
     (pin "3")
-    (pin "4")
-    (pin "5")
     (pin "6")
     (pin "7")
@@
     )
   )
-  (symbol (lib_id "TC20-11SRWA:TC20-11SRWA") (at 257.81 53.34 270) (unit 1)
+  (symbol (lib_name "TC20-11SRWA_2") (lib_id "TC20-11SRWA:TC20-11SRWA") (at 257.81 53.34 270) (unit 1)
     (in_bom yes) (on_board yes) (dnp no)
-    (property "Reference" "D2" (at 271.78 64.77 90)
+    (property "Reference" "D2" (at 250.19 64.77 90)
       (effects (font (size 1.27 1.27)) (justify right))
     )
-    (property "Value" "TC20-11SRWA" (at 246.38 58.42 0)
+    (property "Value" "TC20-11SRWA" (at 246.38 57.15 0)
       (effects (font (size 1.27 1.27)) (justify right))
     )
@@
     (pin "2")
     (pin "3")
-    (pin "4")
-    (pin "5")
     (pin "6")
     (pin "7")
@@
     )
   )
-  (symbol (lib_id "TC20-11SRWA:TC20-11SRWA") (at 173.99 53.34 270) (unit 1)
+  (symbol (lib_name "TC20-11SRWA_5") (lib_id "TC20-11SRWA:TC20-11SRWA") (at 173.99 53.34 270) (unit 1)
     (in_bom yes) (on_board yes) (dnp no)
-    (property "Reference" "D5" (at 187.96 64.77 90)
+    (property "Reference" "D5" (at 166.37 64.77 90)
       (effects (font (size 1.27 1.27)) (justify right))
     )
-    (property "Value" "TC20-11SRWA" (at 162.56 58.42 0)
+    (property "Value" "TC20-11SRWA" (at 162.56 57.15 0)
       (effects (font (size 1.27 1.27)) (justify right))
     )
-    (property "Footprint" "TC20-11SRWA:LED_TC20-11SRWA" (at 173.99 53.34 0)
+    (property "Footprint" "TC20-11SRWA:LED_TC20-11SRWA" (at 184.15 53.34 0)
       (effects (font (size 1.27 1.27)) (justify bottom) hide)
     )
@@
       (effects (font (size 1.27 1.27)) (justify bottom) hide)
     )
-    (property "Description" "\nDot Matrix Display Module 5 x 7 Common Anode Row, Common Cathode Column Red 1.85V - 1.50 L x 2.09 W x 0.33 H (38.10mm x 53.10mm x 8.50mm)\n" (at 173.99 53.34 0)
+    (property "Description" "\nDot Matrix Display Module 5 x 7 Common Anode Row, Common Cathode Column Red 1.85V - 1.50 L x 2.09 W x 0.33 H (38.10mm x 53.10mm x 8.50mm)\n" (at 161.29 53.34 0)
       (effects (font (size 1.27 1.27)) (justify bottom) hide)
     )
@@
     (pin "2")
     (pin "3")
-    (pin "4")
-    (pin "5")
     (pin "6")
     (pin "7")
@@
     )
   )
-  (symbol (lib_id "TC20-11SRWA:TC20-11SRWA") (at 201.93 53.34 270) (unit 1)
+  (symbol (lib_name "TC20-11SRWA_4") (lib_id "TC20-11SRWA:TC20-11SRWA") (at 201.93 53.34 270) (unit 1)
     (in_bom yes) (on_board yes) (dnp no)
-    (property "Reference" "D4" (at 215.9 64.77 90)
+    (property "Reference" "D4" (at 194.31 64.77 90)
       (effects (font (size 1.27 1.27)) (justify right))
     )
-    (property "Value" "TC20-11SRWA" (at 190.5 58.42 0)
+    (property "Value" "TC20-11SRWA" (at 190.5 57.15 0)
       (effects (font (size 1.27 1.27)) (justify right))
     )
@@
     (pin "2")
     (pin "3")
-    (pin "4")
-    (pin "5")
     (pin "6")
     (pin "7")
@@
   (symbol (lib_id "TC20-11SRWA:TC20-11SRWA") (at 146.05 53.34 270) (unit 1)
     (in_bom yes) (on_board yes) (dnp no)
-    (property "Reference" "D6" (at 160.02 64.77 90)
+    (property "Reference" "D6" (at 138.43 64.77 90)
       (effects (font (size 1.27 1.27)) (justify right))
     )
-    (property "Value" "TC20-11SRWA" (at 134.62 58.42 0)
+    (property "Value" "TC20-11SRWA" (at 134.62 57.15 0)
       (effects (font (size 1.27 1.27)) (justify right))
     )
@@
     (pin "2")
     (pin "3")
-    (pin "4")
-    (pin "5")
     (pin "6")
     (pin "7")
@@
     )
   )
-  (symbol (lib_id "TC20-11SRWA:TC20-11SRWA") (at 229.87 53.34 270) (unit 1)
+  (symbol (lib_name "TC20-11SRWA_3") (lib_id "TC20-11SRWA:TC20-11SRWA") (at 229.87 53.34 270) (unit 1)
     (in_bom yes) (on_board yes) (dnp no)
-    (property "Reference" "D3" (at 243.84 64.77 90)
+    (property "Reference" "D3" (at 222.25 64.77 90)
       (effects (font (size 1.27 1.27)) (justify right))
     )
-    (property "Value" "TC20-11SRWA" (at 218.44 58.42 0)
+    (property "Value" "TC20-11SRWA" (at 218.44 57.15 0)
       (effects (font (size 1.27 1.27)) (justify right))
     )
@@
     (pin "2")
     (pin "3")
-    (pin "4")
-    (pin "5")
     (pin "6")
     (pin "7")
